File: conn.kicad_sch (KiCad schematic)
At the start: 11 parts, among them J7 6100.3300.33

Commit message: Updated BoM
Parts:
- removed F2: 3A, symbol Device:Fuse
- added TB-F2: 1880410000, symbol Device:Fuse
- FH1: Cost (none) -> $6.16; Mfr (none) -> Littelfuse Inc.
- J7: Cost (none) -> $15.18
- LED3: Cost (none) -> $0.44; Mfr (none) -> TT Electronics
- PS1: Cost (none) -> $138.29
- PTJP5: Cost (none) -> $0.69; Mfr (none) -> Phoenix Contact
- TB-F1: renamed from F1; value 1A -> 1880410000; Cost (none) -> $33.68; Info (none) -> 1A; Mfr (none) -> Weidmüller
- TB1, TB2, TB3, TB4: Cost (none) -> $1.83
Connections:
- net 24VDC2: now also TB-F2.2
- net at TB4. (D): now also PTJP5.2
- net at PS1.2.2 (+): now also TB-F2.1
Other:
- moved on the sheet: TB-F1

Commit message: Updated PB SW Part#
Parts:
- renumbered TB-F1 to F1
Connections:
- net at TB4. (D): now also PTJP5.2
Changed lines of the file:
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@@
+				)
+			)
+			(project "3xCarbide Permit ILK"
+				(path "/224bdcb2-225d-496a-8b41-82b301326953"
+					(reference "TB-F2")
+					(unit 1)
 				)
 			)
@@
 		(in_pos_files yes)
 		(dnp no)
-		(property "Reference" "TB-F1"
+		(property "Reference" "F1"
 			(at 152.4 161.036 90)
 			(show_name no)

Commit message: Added DRFT
Connections:
- net at TB4. (D): now also PTJP5.2
Changed lines of the file:
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@@
 		(comment 1 "ENGR: J.Park")
 		(comment 2 "CHKR: J.P")
+		(comment 3 "DRFT: KiCad v10")
 	)
 	(circle

Commit message: Added accessary
Parts:
- added EDP1: 3208375, symbol JP_3xCarbide:TB-End
- renumbered F1 to TB-F1
Connections:
- net at TB4. (D): now also PTJP5.2
Other:
- note added: "0.00"
- note added: "Related accessories"

Commit message: Update PB with Honeywell 2PB11
Parts:
- renumbered TB-F1 to F1
Connections:
- net at TB4. (D): now also PTJP5.2
Changed lines of the file:
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@@
+				)
+			)
+			(project "3xCarbide Permit ILK"
+				(path "/224bdcb2-225d-496a-8b41-82b301326953"
+					(reference "EDP1")
+					(unit 1)
 				)
 			)
@@
 		(in_pos_files yes)
 		(dnp no)
-		(property "Reference" "TB-F1"
+		(property "Reference" "F1"
 			(at 152.4 161.036 90)
 			(show_name no)
