File: conn.kicad_sch (KiCad schematic)
At the start: 17 parts, among them J7 6100.3300.33

Commit message: updated 3input-SSR Lib
Connections:
- net at TB4. (D): now also PTJP5.2
Changed lines of the file:
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@@
 		)
 		(instances
+			(project ".kicad_sch"
+				(path "/09dbfdd6-7cc7-4520-a5d9-a383f63872a0/224bdcb2-225d-496a-8b41-82b301326953"
+					(reference "Acc.Socket1")
+					(unit 1)
+				)
+			)
 			(project "3xCarbide Permit ILK"
 				(path "/224bdcb2-225d-496a-8b41-82b301326953"
@@
 		)
 		(instances
+			(project ".kicad_sch"
+				(path "/09dbfdd6-7cc7-4520-a5d9-a383f63872a0/224bdcb2-225d-496a-8b41-82b301326953"
+					(reference "Acc.PLUG")
+					(unit 1)
+				)
+			)
 			(project "3xCarbide Permit ILK"
 				(path "/224bdcb2-225d-496a-8b41-82b301326953"
@@
 		)
 		(instances
+			(project ".kicad_sch"
+				(path "/09dbfdd6-7cc7-4520-a5d9-a383f63872a0/224bdcb2-225d-496a-8b41-82b301326953"
+					(reference "R6")
+					(unit 1)
+				)
+			)
 			(project "3xCarbide Permit ILK"
 				(path "/224bdcb2-225d-496a-8b41-82b301326953"
@@
 		)
 		(instances
+			(project ".kicad_sch"
+				(path "/09dbfdd6-7cc7-4520-a5d9-a383f63872a0/224bdcb2-225d-496a-8b41-82b301326953"
+					(reference "Acc.Bcksh1")
+					(unit 1)
+				)
+			)
 			(project "3xCarbide Permit ILK"
 				(path "/224bdcb2-225d-496a-8b41-82b301326953"
@@
 		)
 		(instances
+			(project ".kicad_sch"
+				(path "/09dbfdd6-7cc7-4520-a5d9-a383f63872a0/224bdcb2-225d-496a-8b41-82b301326953"
+					(reference "PTJP6")
+					(unit 1)
+				)
+			)
 			(project "3xCarbide Permit ILK"
 				(path "/224bdcb2-225d-496a-8b41-82b301326953"
@@
 		)
 		(instances
+			(project ".kicad_sch"
+				(path "/09dbfdd6-7cc7-4520-a5d9-a383f63872a0/224bdcb2-225d-496a-8b41-82b301326953"
+					(reference "Acc.PIN1")
+					(unit 1)
+				)
+			)
 			(project "3xCarbide Permit ILK"
 				(path "/224bdcb2-225d-496a-8b41-82b301326953"
