File: 3xCarbide Permit ILK.kicad_sch (KiCad schematic)
At the start: 43 parts, among them J1 UT00104PH, J2 UT00104PH, J3 UT00104SH, J4 UT00104SH, J5 UT00104SH, J6 UT00104SH, SW1 PB(N.C), SW2 PB(N.C), SW3 PB(N.C), SW4 PB(N.C), SW5 PB(N.C), SW6 PB(N.C)

Commit message: Updated BoM
Parts:
- J1, J2: Cost (none) -> $22.73
- J3, J4, J5, J6: Cost (none) -> $24.98
- LED1, LED2, LED4, LED5, LED6: Cost (none) -> $0.44; Mfr (none) -> TT Electronics
- PTJP1, PTJP2, PTJP3, PTJP4: Cost (none) -> $0.69; Mfr (none) -> Phoenix Contact
- SSR-A0, SSR-A1, SSR-A2, SSR-A3, SSR-B0, SSR-B1, SSR-B2, SSR-B3: Cost (none) -> $63
- TB-A1, TB-A2, TB-A3, TB-A4, TB-B1, TB-B2, TB-B3, TB-B4: Cost (none) -> $1.83
Connections:
- net at J2. (D): no longer TB-B1. (D)
- net at DPM1.1 (CN5): now also LED4.2 (A), SSR-StsA1.1
- net at J1. (D): now also TB-A3. (D)
- net at DPM3.1 (CN5): now also LED6.2 (A), SSR-StsA3.1
- net at J4. (D): now also DPM2.4 (CN2)
- net at J5. (D): now also SSR-A3.13
- new net: J2. (D), TB-B1. (D)
- new net: J1. (D), TB-A1. (D)
- new net: J2. (D), TB-B3. (D)
- now unconnected: J2. (D)

Commit message: Updated PB SW Part#
Parts:
- SW1, SW2, SW3, SW4, SW5, SW6: value PB(N.C) -> 18535CD; Cost (none) -> $12.96; Mfr (none) -> APEM Inc.
Connections:
- net at J2. (D): no longer TB-B1. (D)
- net at DPM1.1 (CN5): now also LED4.2 (A), SSR-StsA1.1
- net at J1. (D): now also TB-A3. (D)
- net at DPM3.1 (CN5): now also LED6.2 (A), SSR-StsA3.1
- net at J4. (D): now also DPM2.4 (CN2)
- net at J5. (D): now also SSR-A3.13
- new net: J2. (D), TB-B1. (D)
- new net: J1. (D), TB-A1. (D)
- new net: J2. (D), TB-B3. (D)
- now unconnected: J2. (D)
Changed lines of the file:
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@@
 			)
 		)
-		(property "Value" "PB(N.C)"
+		(property "Value" "18535CD"
 			(at 143.51 123.19 0)
 			(show_name no)
@@
 			)
 		)
-		(property "Description" "Push button switch, push-to-open, generic, two pins"
+		(property "Description" "SWITCH PUSH SPDT 0.1A 30V, Electrical Life 60,000 Cycles, 100 mA(DC)"
 			(at 143.51 120.65 0)
 			(hide yes)
@@
 			)
 		)
-		(property "Mfr" ""
+		(property "Mfr" "APEM Inc."
 			(at 143.51 120.65 0)
 			(hide yes)
@@
 			)
 		)
+		(property "Cost" "$12.96"
+			(at 143.51 120.65 0)
+			(hide yes)
+			(show_name no)
+			(do_not_autoplace no)
+			(effects
+				(font
+					(size 1.27 1.27)
+				)
+			)
+		)
 		(pin "1"
 		)
@@
 			)
 		)
-		(property "Value" "PB(N.C)"
+		(property "Value" "18535CD"
 			(at 142.24 73.66 0)
 			(show_name no)
@@
 			)
 		)
-		(property "Description" "Push button switch, push-to-open, generic, two pins"
+		(property "Description" "SWITCH PUSH SPDT 0.1A 30V, Electrical Life 60,000 Cycles, 100 mA(DC)"
 			(at 142.24 71.12 0)
 			(hide yes)
@@
 			)
 		)
-		(property "Mfr" ""
+		(property "Mfr" "APEM Inc."
 			(at 142.24 71.12 0)
 			(hide yes)
@@
 			)
 		)
+		(property "Cost" "$12.96"
+			(at 142.24 71.12 0)
+			(hide yes)
+			(show_name no)
+			(do_not_autoplace no)
+			(effects
+				(font
+					(size 1.27 1.27)
+				)
+			)
+		)
 		(pin "1"
 		)
@@
 			)
 		)
-		(property "Value" "PB(N.C)"
+		(property "Value" "18535CD"
 			(at 143.51 143.51 0)
 			(show_name no)
@@
 			)
 		)
-		(property "Description" "Push button switch, push-to-open, generic, two pins"
+		(property "Description" "SWITCH PUSH SPDT 0.1A 30V, Electrical Life 60,000 Cycles, 100 mA(DC)"
 			(at 143.51 140.97 0)
 			(hide yes)
@@
 			)
 		)
-		(property "Mfr" ""
+		(property "Mfr" "APEM Inc."
 			(at 143.51 140.97 0)
 			(hide yes)
@@
 			)
 		)
+		(property "Cost" "$12.96"
+			(at 143.51 140.97 0)
+			(hide yes)
+			(show_name no)
+			(do_not_autoplace no)
+			(effects
+				(font
+					(size 1.27 1.27)
+				)
+			)
+		)
 		(pin "1"
 		)
@@
 			)
 		)
-		(property "Value" "PB(N.C)"
+		(property "Value" "18535CD"
 			(at 142.24 53.34 0)
 			(show_name no)
@@
 			)
 		)
-		(property "Description" "Push button switch, push-to-open, generic, two pins"
+		(property "Description" "SWITCH PUSH SPDT 0.1A 30V, Electrical Life 60,000 Cycles, 100 mA(DC)"
 			(at 142.24 50.8 0)
 			(hide yes)
@@
 			)
 		)
-		(property "Mfr" ""
+		(property "Mfr" "APEM Inc."
 			(at 142.24 50.8 0)
 			(hide yes)
@@
 			)
 		)
+		(property "Cost" "$12.96"
+			(at 142.24 50.8 0)
+			(hide yes)
+			(show_name no)
+			(do_not_autoplace no)
+			(effects
+				(font
+					(size 1.27 1.27)
+				)
+			)
+		)
 		(pin "1"
 		)
@@
 			)
 		)
-		(property "Value" "PB(N.C)"
+		(property "Value" "18535CD"
 			(at 144.78 212.09 0)
 			(show_name no)
@@
 			)
 		)
-		(property "Description" "Push button switch, push-to-open, generic, two pins"
+		(property "Description" "SWITCH PUSH SPDT 0.1A 30V, Electrical Life 60,000 Cycles, 100 mA(DC)"
 			(at 144.78 209.55 0)
 			(hide yes)
@@
 			)
 		)
-		(property "Mfr" ""
+		(property "Mfr" "APEM Inc."
 			(at 144.78 209.55 0)
 			(hide yes)
@@
 			)
 		)
+		(property "Cost" "$12.96"
+			(at 144.78 209.55 0)
+			(hide yes)
+			(show_name no)
+			(do_not_autoplace no)
+			(effects
+				(font
+					(size 1.27 1.27)
+				)
+			)
+		)
 		(pin "1"
 		)
@@
 			)
 		)
-		(property "Value" "PB(N.C)"
+		(property "Value" "18535CD"
 			(at 144.78 191.77 0)
 			(show_name no)
@@
 			)
 		)
-		(property "Description" "Push button switch, push-to-open, generic, two pins"
+		(property "Description" "SWITCH PUSH SPDT 0.1A 30V, Electrical Life 60,000 Cycles, 100 mA(DC)"
 			(at 144.78 189.23 0)
 			(hide yes)
@@
 			)
 		)
-		(property "Mfr" ""
+		(property "Mfr" "APEM Inc."
 			(at 144.78 189.23 0)
 			(hide yes)
@@
 			)
 		)
+		(property "Cost" "$12.96"
+			(at 144.78 189.23 0)
+			(hide yes)
+			(show_name no)
+			(do_not_autoplace no)
+			(effects
+				(font
+					(size 1.27 1.27)
+				)
+			)
+		)
 		(pin "1"
 		)
@@
 		)
 	)
+	(embedded_fonts no)
 )

Commit message: Added DRFT
Connections:
- net at J2. (D): no longer TB-B1. (D)
- net at DPM1.1 (CN5): now also LED4.2 (A), SSR-StsA1.1
- net at J1. (D): now also TB-A3. (D)
- net at DPM3.1 (CN5): now also LED6.2 (A), SSR-StsA3.1
- net at J4. (D): now also DPM2.4 (CN2)
- net at J5. (D): now also SSR-A3.13
- new net: J2. (D), TB-B1. (D)
- new net: J1. (D), TB-A1. (D)
- new net: J2. (D), TB-B3. (D)
- now unconnected: J2. (D)
Changed lines of the file:
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@@
 		(company "SLAC")
 		(comment 1 "ENGR: J.Park")
-		(comment 2 "CHKR: J.P")
+		(comment 2 "CHKR: J.Park")
+		(comment 3 "DRFT: KiCad v10")
 	)
 	(rectangle

Commit message: Added accessary
Connections:
- net at J2. (D): no longer TB-B1. (D)
- net at DPM1.1 (CN5): now also LED4.2 (A), SSR-StsA1.1
- net at J1. (D): now also TB-A3. (D)
- net at DPM3.1 (CN5): now also LED6.2 (A), SSR-StsA3.1
- net at J4. (D): now also DPM2.4 (CN2)
- net at J5. (D): now also SSR-A3.13
- new net: J2. (D), TB-B1. (D)
- new net: J1. (D), TB-A1. (D)
- new net: J2. (D), TB-B3. (D)
- now unconnected: J2. (D)
Changed lines of the file:
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@@
 		)
 	)
-	(embedded_fonts no)
 )

Commit message: Update PB with Honeywell 2PB11
Parts:
- SW1, SW2, SW3, SW4, SW5, SW6: value 18535CD -> 2PB11; Cost $12.96 -> $165.16; Mfr APEM Inc. -> Honeywell Sensing
Connections:
- net at J2. (D): no longer TB-B1. (D)
- net at DPM1.1 (CN5): now also LED4.2 (A), SSR-StsA1.1
- net at J1. (D): now also TB-A3. (D)
- net at DPM3.1 (CN5): now also LED6.2 (A), SSR-StsA3.1
- net at J4. (D): now also DPM2.4 (CN2)
- net at J5. (D): now also SSR-A3.13
- new net: J2. (D), TB-B1. (D)
- new net: J1. (D), TB-A1. (D)
- new net: J2. (D), TB-B3. (D)
- now unconnected: J2. (D)
Changed lines of the file:
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@@
 			)
 		)
-		(property "Value" "18535CD"
+		(property "Value" "2PB11"
 			(at 143.51 123.19 0)
 			(show_name no)
@@
 			)
 		)
-		(property "Datasheet" ""
+		(property "Datasheet" "https://www.digikey.com/en/products/detail/honeywell-sensing-and-productivity-solutions/2PB11/1248816"
 			(at 143.51 115.57 0)
 			(hide yes)
@@
 			)
 		)
-		(property "Description" "SWITCH PUSH SPDT 0.1A 30V, Electrical Life 60,000 Cycles, 100 mA(DC)"
+		(property "Description" "PB Switch SPDT x 2 Standard Panel Mount, Rear"
 			(at 143.51 120.65 0)
 			(hide yes)
@@
 			)
 		)
-		(property "Mfr" "APEM Inc."
+		(property "Mfr" "Honeywell Sensing"
 			(at 143.51 120.65 0)
 			(hide yes)
@@
 			)
 		)
-		(property "Cost" "$12.96"
+		(property "Cost" "$165.16"
 			(at 143.51 120.65 0)
 			(hide yes)
@@
 			)
 		)
-		(property "Value" "18535CD"
+		(property "Value" "2PB11"
 			(at 142.24 73.66 0)
 			(show_name no)
@@
 			)
 		)
-		(property "Datasheet" ""
+		(property "Datasheet" "https://www.digikey.com/en/products/detail/honeywell-sensing-and-productivity-solutions/2PB11/1248816"
 			(at 142.24 66.04 0)
 			(hide yes)
@@
 			)
 		)
-		(property "Description" "SWITCH PUSH SPDT 0.1A 30V, Electrical Life 60,000 Cycles, 100 mA(DC)"
+		(property "Description" "PB Switch SPDT x 2 Standard Panel Mount, Rear"
 			(at 142.24 71.12 0)
 			(hide yes)
@@
 			)
 		)
-		(property "Mfr" "APEM Inc."
+		(property "Mfr" "Honeywell Sensing"
 			(at 142.24 71.12 0)
 			(hide yes)
@@
 			)
 		)
-		(property "Cost" "$12.96"
+		(property "Cost" "$165.16"
 			(at 142.24 71.12 0)
 			(hide yes)
@@
 			)
 		)
-		(property "Value" "18535CD"
+		(property "Value" "2PB11"
 			(at 143.51 143.51 0)
 			(show_name no)
@@
 			)
 		)
-		(property "Datasheet" ""
+		(property "Datasheet" "https://www.digikey.com/en/products/detail/honeywell-sensing-and-productivity-solutions/2PB11/1248816"
 			(at 143.51 135.89 0)
 			(hide yes)
@@
 			)
 		)
-		(property "Description" "SWITCH PUSH SPDT 0.1A 30V, Electrical Life 60,000 Cycles, 100 mA(DC)"
+		(property "Description" "PB Switch SPDT x 2 Standard Panel Mount, Rear"
 			(at 143.51 140.97 0)
 			(hide yes)
@@
 			)
 		)
-		(property "Mfr" "APEM Inc."
+		(property "Mfr" "Honeywell Sensing"
 			(at 143.51 140.97 0)
 			(hide yes)
@@
 			)
 		)
-		(property "Cost" "$12.96"
+		(property "Cost" "$165.16"
 			(at 143.51 140.97 0)
 			(hide yes)
@@
 			)
 		)
-		(property "Value" "18535CD"
+		(property "Value" "2PB11"
 			(at 142.24 53.34 0)
 			(show_name no)
@@
 			)
 		)
-		(property "Datasheet" ""
+		(property "Datasheet" "https://www.digikey.com/en/products/detail/honeywell-sensing-and-productivity-solutions/2PB11/1248816"
 			(at 142.24 45.72 0)
 			(hide yes)
@@
 			)
 		)
-		(property "Description" "SWITCH PUSH SPDT 0.1A 30V, Electrical Life 60,000 Cycles, 100 mA(DC)"
+		(property "Description" "PB Switch SPDT x 2 Standard Panel Mount, Rear"
 			(at 142.24 50.8 0)
 			(hide yes)
@@
 			)
 		)
-		(property "Mfr" "APEM Inc."
+		(property "Mfr" "Honeywell Sensing"
 			(at 142.24 50.8 0)
 			(hide yes)
@@
 			)
 		)
-		(property "Cost" "$12.96"
+		(property "Cost" "$165.16"
 			(at 142.24 50.8 0)
 			(hide yes)
@@
 			)
 		)
-		(property "Value" "18535CD"
+		(property "Value" "2PB11"
 			(at 144.78 212.09 0)
 			(show_name no)
@@
 			)
 		)
-		(property "Datasheet" ""
+		(property "Datasheet" "https://www.digikey.com/en/products/detail/honeywell-sensing-and-productivity-solutions/2PB11/1248816"
 			(at 144.78 204.47 0)
 			(hide yes)
@@
 			)
 		)
-		(property "Description" "SWITCH PUSH SPDT 0.1A 30V, Electrical Life 60,000 Cycles, 100 mA(DC)"
+		(property "Description" "PB Switch SPDT x 2 Standard Panel Mount, Rear"
 			(at 144.78 209.55 0)
 			(hide yes)
@@
 			)
 		)
-		(property "Mfr" "APEM Inc."
+		(property "Mfr" "Honeywell Sensing"
 			(at 144.78 209.55 0)
 			(hide yes)
@@
 			)
 		)
-		(property "Cost" "$12.96"
+		(property "Cost" "$165.16"
 			(at 144.78 209.55 0)
 			(hide yes)
@@
 			)
 		)
-		(property "Value" "18535CD"
+		(property "Value" "2PB11"
 			(at 144.78 191.77 0)
 			(show_name no)
@@
 			)
 		)
-		(property "Datasheet" ""
+		(property "Datasheet" "https://www.digikey.com/en/products/detail/honeywell-sensing-and-productivity-solutions/2PB11/1248816"
 			(at 144.78 184.15 0)
 			(hide yes)
@@
 			)
 		)
-		(property "Description" "SWITCH PUSH SPDT 0.1A 30V, Electrical Life 60,000 Cycles, 100 mA(DC)"
+		(property "Description" "PB Switch SPDT x 2 Standard Panel Mount, Rear"
 			(at 144.78 189.23 0)
 			(hide yes)
@@
 			)
 		)
-		(property "Mfr" "APEM Inc."
+		(property "Mfr" "Honeywell Sensing"
 			(at 144.78 189.23 0)
 			(hide yes)
@@
 			)
 		)
-		(property "Cost" "$12.96"
+		(property "Cost" "$165.16"
 			(at 144.78 189.23 0)
 			(hide yes)
@@
 		)
 	)
+	(embedded_fonts no)
 )

Commit message: Update Murre SSR 52511 vendor
Parts:
- SSR-A0, SSR-A1, SSR-A2, SSR-A3, SSR-B0, SSR-B1, SSR-B2, SSR-B3: Cost $63 -> $22.50
Connections:
- net at J2. (D): no longer TB-B1. (D)
- net at DPM1.1 (CN5): now also LED4.2 (A), SSR-StsA1.1
- net at J1. (D): now also TB-A3. (D)
- net at DPM3.1 (CN5): now also LED6.2 (A), SSR-StsA3.1
- net at J4. (D): now also DPM2.4 (CN2)
- net at J5. (D): now also SSR-A3.13
- new net: J2. (D), TB-B1. (D)
- new net: J1. (D), TB-A1. (D)
- new net: J2. (D), TB-B3. (D)
- now unconnected: J2. (D)
Changed lines of the file:
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@@
 			)
 		)
-		(property "Datasheet" "https://www.mouser.com/datasheet/3/5927/2/52511_Product_PDF_en.pdf"
+		(property "Datasheet" "https://www.automationdirect.com/adc/shopping/catalog/relays_-z-_timers/optocoupler_relays/52511?srsltid=AfmBOoq-n2697LSqzmjaMwd-Sr5CC2yJvxaUk5WAfUlPuLUUbm9nKA0Z"
 			(at 161.798 153.924 0)
 			(hide yes)
@@
 			)
 		)
-		(property "Description" "MIRO TR 24VDC 20KHZ IN<1MA OPTO-"
+		(property "Description" "MIRO TR 24VDC 20KHZ IN<1MA OPTO-SPST"
 			(at 162.814 151.638 0)
 			(hide yes)
@@
 			)
 		)
-		(property "Cost" "$63"
+		(property "Cost" "$22.50"
 			(at 153.67 146.05 0)
 			(hide yes)
@@
 			)
 		)
-		(property "Datasheet" "https://www.mouser.com/datasheet/3/5927/2/52511_Product_PDF_en.pdf"
+		(property "Datasheet" "https://www.automationdirect.com/adc/shopping/catalog/relays_-z-_timers/optocoupler_relays/52511?srsltid=AfmBOoq-n2697LSqzmjaMwd-Sr5CC2yJvxaUk5WAfUlPuLUUbm9nKA0Z"
 			(at 310.388 211.074 0)
 			(hide yes)
@@
 			)
 		)
-		(property "Description" "MIRO TR 24VDC 20KHZ IN<1MA OPTO-"
+		(property "Description" "MIRO TR 24VDC 20KHZ IN<1MA OPTO-SPST"
 			(at 311.404 208.788 0)
 			(hide yes)
@@
 			)
 		)
-		(property "Cost" "$63"
+		(property "Cost" "$22.50"
 			(at 302.26 203.2 0)
 			(hide yes)
@@
 			)
 		)
-		(property "Datasheet" "https://www.mouser.com/datasheet/3/5927/2/52511_Product_PDF_en.pdf"
+		(property "Datasheet" "https://www.automationdirect.com/adc/shopping/catalog/relays_-z-_timers/optocoupler_relays/52511?srsltid=AfmBOoq-n2697LSqzmjaMwd-Sr5CC2yJvxaUk5WAfUlPuLUUbm9nKA0Z"
 			(at 161.798 133.604 0)
 			(hide yes)
@@
 			)
 		)
-		(property "Description" "MIRO TR 24VDC 20KHZ IN<1MA OPTO-"
+		(property "Description" "MIRO TR 24VDC 20KHZ IN<1MA OPTO-SPST"
 			(at 162.814 131.318 0)
 			(hide yes)
@@
 			)
 		)
-		(property "Cost" "$63"
+		(property "Cost" "$22.50"
 			(at 153.67 125.73 0)
 			(hide yes)
@@
 			)
 		)
-		(property "Datasheet" "https://www.mouser.com/datasheet/3/5927/2/52511_Product_PDF_en.pdf"
+		(property "Datasheet" "https://www.automationdirect.com/adc/shopping/catalog/relays_-z-_timers/optocoupler_relays/52511?srsltid=AfmBOoq-n2697LSqzmjaMwd-Sr5CC2yJvxaUk5WAfUlPuLUUbm9nKA0Z"
 			(at 160.528 63.754 0)
 			(hide yes)
@@
 			)
 		)
-		(property "Description" "MIRO TR 24VDC 20KHZ IN<1MA OPTO-"
+		(property "Description" "MIRO TR 24VDC 20KHZ IN<1MA OPTO-SPST"
 			(at 161.544 61.468 0)
 			(hide yes)
@@
 			)
 		)
-		(property "Cost" "$63"
+		(property "Cost" "$22.50"
 			(at 152.4 55.88 0)
 			(hide yes)
@@
 			)
 		)
-		(property "Datasheet" "https://www.mouser.com/datasheet/3/5927/2/52511_Product_PDF_en.pdf"
+		(property "Datasheet" "https://www.automationdirect.com/adc/shopping/catalog/relays_-z-_timers/optocoupler_relays/52511?srsltid=AfmBOoq-n2697LSqzmjaMwd-Sr5CC2yJvxaUk5WAfUlPuLUUbm9nKA0Z"
 			(at 160.528 84.074 0)
 			(hide yes)
@@
 			)
 		)
-		(property "Description" "MIRO TR 24VDC 20KHZ IN<1MA OPTO-"
+		(property "Description" "MIRO TR 24VDC 20KHZ IN<1MA OPTO-SPST"
 			(at 161.544 81.788 0)
 			(hide yes)
@@
 			)
 		)
-		(property "Cost" "$63"
+		(property "Cost" "$22.50"
 			(at 152.4 76.2 0)
 			(hide yes)
@@
 			)
 		)
-		(property "Datasheet" "https://www.mouser.com/datasheet/3/5927/2/52511_Product_PDF_en.pdf"
+		(property "Datasheet" "https://www.automationdirect.com/adc/shopping/catalog/relays_-z-_timers/optocoupler_relays/52511?srsltid=AfmBOoq-n2697LSqzmjaMwd-Sr5CC2yJvxaUk5WAfUlPuLUUbm9nKA0Z"
 			(at 163.068 222.504 0)
 			(hide yes)
@@
 			)
 		)
-		(property "Description" "MIRO TR 24VDC 20KHZ IN<1MA OPTO-"
+		(property "Description" "MIRO TR 24VDC 20KHZ IN<1MA OPTO-SPST"
 			(at 164.084 220.218 0)
 			(hide yes)
@@
 			)
 		)
-		(property "Cost" "$63"
+		(property "Cost" "$22.50"
 			(at 154.94 214.63 0)
 			(hide yes)
@@
 			)
 		)
-		(property "Datasheet" "https://www.mouser.com/datasheet/3/5927/2/52511_Product_PDF_en.pdf"
+		(property "Datasheet" "https://www.automationdirect.com/adc/shopping/catalog/relays_-z-_timers/optocoupler_relays/52511?srsltid=AfmBOoq-n2697LSqzmjaMwd-Sr5CC2yJvxaUk5WAfUlPuLUUbm9nKA0Z"
 			(at 310.388 190.754 0)
 			(hide yes)
@@
 			)
 		)
-		(property "Description" "MIRO TR 24VDC 20KHZ IN<1MA OPTO-"
+		(property "Description" "MIRO TR 24VDC 20KHZ IN<1MA OPTO-SPST"
 			(at 311.404 188.468 0)
 			(hide yes)
@@
 			)
 		)
-		(property "Cost" "$63"
+		(property "Cost" "$22.50"
 			(at 302.26 182.88 0)
 			(hide yes)
@@
 			)
 		)
-		(property "Datasheet" "https://www.mouser.com/datasheet/3/5927/2/52511_Product_PDF_en.pdf"
+		(property "Datasheet" "https://www.automationdirect.com/adc/shopping/catalog/relays_-z-_timers/optocoupler_relays/52511?srsltid=AfmBOoq-n2697LSqzmjaMwd-Sr5CC2yJvxaUk5WAfUlPuLUUbm9nKA0Z"
 			(at 163.068 202.184 0)
 			(hide yes)
@@
 			)
 		)
-		(property "Description" "MIRO TR 24VDC 20KHZ IN<1MA OPTO-"
+		(property "Description" "MIRO TR 24VDC 20KHZ IN<1MA OPTO-SPST"
 			(at 164.084 199.898 0)
 			(hide yes)
@@
 			)
 		)
-		(property "Cost" "$63"
+		(property "Cost" "$22.50"
 			(at 154.94 194.31 0)
 			(hide yes)

Commit message: Updated Acc. parts
Parts:
- removed J3, J4, J5, J6: UT00104SH, symbol JP_3xCarbide:CONN_UT00104SH(F)
- added J3, J4, J5, J6: UT00104PH, symbol JP_3xCarbide:CONN_UT00104PH(M)
Connections:
- net Loop1Sts: now also J6. (D)
- net Loop2Sts: now also J6. (D)
- net Loop3Sts: now also J6. (D)
- net SEN_PS: now also J6. (D)
- net at J2. (D): no longer TB-B1. (D)
- net at DPM1.1 (CN5): now also LED4.2 (A), SSR-StsA1.1
- net at DPM1.4 (CN2): now also J3. (D)
- net at J1. (D): now also TB-A3. (D)
- net at SSR-A2.13: now also J4. (D)
- net at SSR-A1.13: now also J3. (D)
- net at DPM3.1 (CN5): now also LED6.2 (A), SSR-StsA3.1
- net at DPM3.4 (CN2): now also J5. (D)
- net at DPM2.4 (CN2): now also J4. (D)
- net at SSR-A3.13: now also J5. (D)
- new net: J2. (D), TB-B1. (D)
- new net: J1. (D), TB-A1. (D)
- new net: J2. (D), TB-B3. (D)
- now unconnected: J2. (D)
Other:
- note added: "To PLC / EPICS"
- note removed: "Permit Loop Status To PLC / EPICS"

Commit message: Edit Permit Loop#
Parts:
- J4: Conn Info Permit Loop#1 -> Permit Loop#2
- J5: Conn Info Permit Loop#1 -> Permit Loop#3
Connections:
- net at J2. (D): no longer TB-B1. (D)
- net at DPM1.1 (CN5): now also LED4.2 (A), SSR-StsA1.1
- net at J1. (D): now also TB-A3. (D)
- net at DPM3.1 (CN5): now also LED6.2 (A), SSR-StsA3.1
- net at J4. (D): now also DPM2.4 (CN2)
- net at J5. (D): now also SSR-A3.13
- new net: J2. (D), TB-B1. (D)
- new net: J1. (D), TB-A1. (D)
- new net: J2. (D), TB-B3. (D)
- now unconnected: J2. (D)
Changed lines of the file:
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@@
 			)
 		)
-		(property "Conn Info" "Permit Loop#1"
+		(property "Conn Info" "Permit Loop#2"
 			(at 227.33 132.08 0)
 			(show_name no)
@@
 			)
 		)
-		(property "Conn Info" "Permit Loop#1"
+		(property "Conn Info" "Permit Loop#3"
 			(at 228.6 200.66 0)
 			(show_name no)
